Commit message: resolved an error with grasping _frame

File: urdf/seven_DOF_arm.xacro (robot description, xacro)
@@ -117,5 +117,5 @@
 	       <box size="0.1 0.1 0.1" />
       </geometry>
-      </collision>>
+      </collision>
 	<xacro:inertial_matrix mass="1"/>
   </link>
@@ -391,7 +391,5 @@
         <origin xyz="0 0 0"/>
         <geometry>
-					<!--
           <box size="${grasp_frame_len} ${grasp_frame_width} ${grasp_frame_height}" />
-					-->
         </geometry>
         <material name="White" />
