Commit message: removed DarkGray as material color

File: urdf/wheel.urdf.xacro (robot description, xacro)
@@ -16,5 +16,5 @@
           <cylinder length="${wheel_height}" radius="${wheel_radius}" />
         </geometry>
-        <material name="DarkGray" />
+        <material name="Black" />
       </visual>
       <collision>
